File: frontend.kicad_sch (KiCad schematic)
At the start: 33 parts, among them U4 PN5120A0HN1, X1 27.12MHz

Commit message: new stuff
Parts:
- renumbered R14 to R12, R15 to R13, R16 to R14, R17 to R15, R18 to R16, R19 to R17, R20 to R18, R21 to R19, R22 to R20, R23 to R21, R24 to R22, R25 to R23, R26 to R24
Other:
- note added: "NFC FRONTEND"
Changed lines of the file:
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@@
 		)
 	)
+	(text "NFC FRONTEND"
+		(exclude_from_sim no)
+		(at 176.53 20.32 0)
+		(effects
+			(font
+				(size 2.54 2.54)
+			)
+		)
+	)
 	(junction
 		(at 130.81 78.74)
@@
 		(on_board yes)
 		(dnp no)
-		(property "Reference" "R26"
+		(property "Reference" "R24"
 			(at 241.3 92.71 90)
 			(effects
@@
 			(project "rfid-mirror"
 				(path "/d5f40065-105e-4e8c-8462-c47ae46f6394/203b1978-e8cc-4c88-9ca8-867d975a8b14"
-					(reference "R26")
+					(reference "R24")
 					(unit 1)
 				)
@@
 		(on_board yes)
 		(dnp no)
-		(property "Reference" "R16"
+		(property "Reference" "R14"
 			(at 127 64.77 0)
 			(effects
@@
 			(project "rfid-mirror"
 				(path "/d5f40065-105e-4e8c-8462-c47ae46f6394/203b1978-e8cc-4c88-9ca8-867d975a8b14"
-					(reference "R16")
+					(reference "R14")
 					(unit 1)
 				)
@@
 		(on_board yes)
 		(dnp no)
-		(property "Reference" "R24"
+		(property "Reference" "R22"
 			(at 241.3 87.63 90)
 			(effects
@@
 			(project "rfid-mirror"
 				(path "/d5f40065-105e-4e8c-8462-c47ae46f6394/203b1978-e8cc-4c88-9ca8-867d975a8b14"
-					(reference "R24")
+					(reference "R22")
 					(unit 1)
 				)
@@
 		(on_board yes)
 		(dnp no)
-		(property "Reference" "R18"
+		(property "Reference" "R16"
 			(at 238.76 69.85 90)
 			(effects
@@
 			(project "rfid-mirror"
 				(path "/d5f40065-105e-4e8c-8462-c47ae46f6394/203b1978-e8cc-4c88-9ca8-867d975a8b14"
-					(reference "R18")
+					(reference "R16")
 					(unit 1)
 				)
@@
 		(on_board yes)
 		(dnp no)
-		(property "Reference" "R21"
+		(property "Reference" "R19"
 			(at 69.85 81.28 90)
 			(effects
@@
 			(project "rfid-mirror"
 				(path "/d5f40065-105e-4e8c-8462-c47ae46f6394/203b1978-e8cc-4c88-9ca8-867d975a8b14"
-					(reference "R21")
+					(reference "R19")
 					(unit 1)
 				)
@@
 		(on_board yes)
 		(dnp no)
-		(property "Reference" "R23"
+		(property "Reference" "R21"
 			(at 69.85 91.44 90)
 			(effects
@@
 			(project "rfid-mirror"
 				(path "/d5f40065-105e-4e8c-8462-c47ae46f6394/203b1978-e8cc-4c88-9ca8-867d975a8b14"
-					(reference "R23")
+					(reference "R21")
 					(unit 1)
 				)
@@
 		(on_board yes)
 		(dnp no)
-		(property "Reference" "R22"
+		(property "Reference" "R20"
 			(at 241.3 85.09 90)
 			(effects
@@
 			(project "rfid-mirror"
 				(path "/d5f40065-105e-4e8c-8462-c47ae46f6394/203b1978-e8cc-4c88-9ca8-867d975a8b14"
-					(reference "R22")
+					(reference "R20")
 					(unit 1)
 				)
@@
 		(on_board yes)
 		(dnp no)
-		(property "Reference" "R15"
+		(property "Reference" "R13"
 			(at 153.67 62.23 0)
 			(effects
@@
 			)
 		)
-		(property "LCSC Part Number" ""
-			(at 148.59 63.5 0)
-			(effects
-				(font
-					(size 1.27 1.27)
-				)
-				(hide yes)
-			)
-		)
 		(pin "1"
 		)
@@
 			(project "rfid-mirror"
 				(path "/d5f40065-105e-4e8c-8462-c47ae46f6394/203b1978-e8cc-4c88-9ca8-867d975a8b14"
-					(reference "R15")
+					(reference "R13")
 					(unit 1)
 				)
@@
 		(dnp no)
 		(fields_autoplaced yes)
-		(property "Reference" "R14"
+		(property "Reference" "R12"
 			(at 203.2 50.7999 0)
 			(effects
@@
 			(project "rfid-mirror"
 				(path "/d5f40065-105e-4e8c-8462-c47ae46f6394/203b1978-e8cc-4c88-9ca8-867d975a8b14"
-					(reference "R14")
+					(reference "R12")
 					(unit 1)
 				)
@@
 		(on_board yes)
 		(dnp no)
-		(property "Reference" "R25"
+		(property "Reference" "R23"
 			(at 241.3 90.17 90)
 			(effects
@@
 			(project "rfid-mirror"
 				(path "/d5f40065-105e-4e8c-8462-c47ae46f6394/203b1978-e8cc-4c88-9ca8-867d975a8b14"
-					(reference "R25")
+					(reference "R23")
 					(unit 1)
 				)
@@
 		(on_board yes)
 		(dnp no)
-		(property "Reference" "R19"
+		(property "Reference" "R17"
 			(at 241.3 80.01 90)
 			(effects
@@
 			(project "rfid-mirror"
 				(path "/d5f40065-105e-4e8c-8462-c47ae46f6394/203b1978-e8cc-4c88-9ca8-867d975a8b14"
-					(reference "R19")
+					(reference "R17")
 					(unit 1)
 				)
@@
 		(on_board yes)
 		(dnp no)
-		(property "Reference" "R20"
+		(property "Reference" "R18"
 			(at 241.3 82.55 90)
 			(effects
@@
 			(project "rfid-mirror"
 				(path "/d5f40065-105e-4e8c-8462-c47ae46f6394/203b1978-e8cc-4c88-9ca8-867d975a8b14"
-					(reference "R20")
+					(reference "R18")
 					(unit 1)
 				)
@@
 		(dnp no)
 		(fields_autoplaced yes)
-		(property "Reference" "R17"
+		(property "Reference" "R15"
 			(at 229.87 66.0399 0)
 			(effects
@@
 			(project ""
 				(path "/d5f40065-105e-4e8c-8462-c47ae46f6394/203b1978-e8cc-4c88-9ca8-867d975a8b14"
-					(reference "R17")
+					(reference "R15")
 					(unit 1)
 				)
