File: mcu.kicad_sch (KiCad schematic)
At the start: 26 parts, among them J2 Conn_ARM_SWD_TagConnect_TC2030, Q2 MMBT3904, Q3 BC860, SW2 B3U-1000P, SW3 1825232, U5 BY25Q128, U6 ESP32-WROOM-32E

Commit message: new stuff
Parts:
- removed Q2: MMBT3904, Package_TO_SOT_SMD:SOT-23, symbol Transistor_BJT:MMBT3904
- removed Q3: BC860, Package_TO_SOT_SMD:SOT-23, symbol Transistor_BJT:BC860
- removed R30, R34: 22R, Resistor_SMD:R_0603_1608Metric, symbol tbraico:22R
- removed R31, R33: 33R, Resistor_SMD:R_0603_1608Metric, symbol tbraico:33R
- removed R35: 10k, Resistor_SMD:R_0603_1608Metric, symbol tbraico:10k
- removed SW3: 1825232, tbraico:1825232, symbol tbraico:1825232-1
- added R28, R31: 220R, Resistor_SMD:R_0603_1608Metric, symbol tbraico:220R
- added R29: 0R, Resistor_SMD:R_0603_1608Metric, symbol tbraico:0R
- added SW3: GF-123-0054, tbraico:SW_GF-123-0054, symbol tbraico:GF-123-0054
- renumbered C25 to C24, C26 to C25, C24 to C26, D5 to D4, D4 to D5, R27 to R25, R28 to R26, R29 to R27, R32 to R30, R36 to R32
Connections:
- net +3V3: now also D4.2 (A); no longer C28.1
- net ESP_BOOTMODE: now also C26.1, C28.2, R27.2, R28.1, SW3.2
- net GND: now also C28.1, R29.1, R31.2
- net at D5.1 (K): now also R31.1
- net at D4.1 (K): now also R28.2
- new net: R29.2, SW3.1
Other:
- moved on the sheet: C24, C25, C26, C27, D4, D5, J2, R27, R30, R32, U5, U6
