File: rfid-mirror.kicad_pcb (KiCad board)
At the start: 2 copper layers, 86.8 x 60.5 mm, 97 parts, among them J1 USB3080-30-01-A, J2 Conn_ARM_SWD_TagConnect_TC2030, Q1 MMBT3904, Q2 MMBT3904, Q3 BC860, SW1 PB400EEQX, SW2 B3U-1000P, SW3 1825232, U1 TPS61291, U2 TPS2116DRL, U3 CP2102N, U4 PN5120A0HN1, U5 BY25Q128, U6 ESP32-WROOM-32E, X1 27.12MHz

Commit message: new stuff
Parts:
- removed Q1, Q2: MMBT3904, Package_TO_SOT_SMD:SOT-23
- removed Q3: BC860, Package_TO_SOT_SMD:SOT-23
- removed the R30 at (110.0, 77.0)
- removed R33: 33R, Resistor_SMD:R_0603_1608Metric
- removed R34: 22R, Resistor_SMD:R_0603_1608Metric
- removed R35: 10k, Resistor_SMD:R_0603_1608Metric
- removed the R5 at (99.6, 63.4)
- removed the R7 at (99.6, 66.5)
- removed the R8 at (103.6, 66.5)
- added R28: 220R, Resistor_SMD:R_0603_1608Metric, F.Cu at (127.0, 68.6)
- added R29: 0R, Resistor_SMD:R_0603_1608Metric, F.Cu at (122.7, 75.5)
- added R4: 220R, Resistor_SMD:R_0603_1608Metric, F.Cu at (103.6, 62.7)
- R31, R6: value 33R -> 220R
- SW3: value 1825232 -> GF-123-0054; footprint tbraico:1825232 -> tbraico:SW_GF-123-0054
- moved R31 18.6 mm to (127.0, 71.1)
- moved D5 14.7 mm to (124.0, 71.1)
- moved D4 11.6 mm to (124.1, 68.6), turned to 180 degrees
- moved SW3 9.25 mm to (113.2, 76.8), turned to 180 degrees
- moved R6 4.00 mm to (99.6, 63.3), turned to -90 degrees
- moved C28 3.23 mm to (117.7, 70.4), turned to 180 degrees
- moved D1 0.75 mm to (103.6, 59.1)
- renumbered C25 to C24, C26 to C25, C24 to C26, D2 to D1, D1 to D2, D5 to D4, D4 to D5, R12 to R10, R13 to R11, R14 to R12, R15 to R13, R16 to R14, R17 to R15, R18 to R16, R19 to R17, R20 to R18, R21 to R19, R22 to R20, R23 to R21, R24 to R22, R25 to R23, R26 to R24, R27 to R25, R28 to R26, R29 to R27, R32 to R30, R36 to R32, R4 to R5, R9 to R7, R10 to R8, R11 to R9
Connections:
- net Net-(D1-A) renamed /ST
- C2 pad 1: /BAT_P -> Net-(CR1-I/O4)
- C26 pad 1: Net-(C24-Pad1) -> /mcu/ESP_BOOTMODE
- C28 pad 1: +3V3 -> GND
- C28 pad 2: Net-(C28-Pad2) -> /mcu/ESP_BOOTMODE
- CR1 pad 5: /BAT_P -> Net-(CR1-I/O4)
- D1 pad 1: Net-(D2-K) -> Net-(D1-K)
- D1 pad 2: Net-(D2-A) -> +3V3
- D2 pad 1: Net-(D1-K) -> Net-(D2-K)
- D4 pad 2: Net-(D5-A) -> +3V3
- D5 pad 1: Net-(D4-K) (its old number) -> Net-(D5-K)
- L1 pad 1: /BAT_P -> Net-(CR1-I/O4)
- R27 pad 2: Net-(C24-Pad1) -> /mcu/ESP_BOOTMODE
- R31 pad 1: Net-(R30-Pad2) -> Net-(D5-K)
- R31 pad 2: Net-(Q2-C) -> GND
- R6 pad 1: Net-(R6-Pad1) -> Net-(D2-K)
- R6 pad 2: Net-(D2-K) -> GND
- SW3 pad 1: /mcu/ESP_BOOTMODE -> Net-(R29-Pad2)
- SW3 pad 2: Net-(C28-Pad2) -> /mcu/ESP_BOOTMODE
- U1 pad 3: /BAT_P -> Net-(CR1-I/O4)
- U1 pad 4: /BAT_P -> Net-(CR1-I/O4)
Routing:
- net Net-(C24-Pad1): track 24.2 -> 0.00 mm
- net /BAT_P: track 29.1 -> 9.19 mm
- net Net-(CR1-I/O4): track 0.00 -> 17.4 mm
- net Net-(C28-Pad2): track 13.3 -> 0.00 mm, vias 2 -> 0
- net /frontend/NFC_IRQ: track 103.7 -> 95.3 mm
- net +3V3: track 188.0 -> 194.4 mm, vias 15 -> 16
- net Net-(R29-Pad2): track 0.00 -> 5.51 mm
- net /mcu/ESP_BOOTMODE: track 66.0 -> 62.2 mm, vias 5 -> 2
- net Net-(Q2-C): track 3.13 -> 0.00 mm
- net Net-(D5-A): track 3.04 -> 0.00 mm
- net /ST: track 20.7 -> 18.1 mm, vias 2 -> 0
- net Net-(D2-A): track 1.99 -> 0.00 mm
- net Net-(R5-Pad1): track 1.53 -> 0.00 mm
- net Net-(D4-K) (its old number): track 1.52 -> 0.00 mm
- net Net-(R6-Pad1): track 1.50 -> 0.00 mm
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Other:
- board text added: "FLASH"
- board text removed: "UART BOOT"
