File: rfid-mirror.kicad_sch (KiCad schematic)
At the start: 38 parts, among them J1 USB3080-30-01-A, Q1 MMBT3904, SW1 PB400EEQX, U1 TPS61291, U2 TPS2116DRL, U3 CP2102N

Commit message: new stuff
Parts:
- removed Q1: MMBT3904, Package_TO_SOT_SMD:SOT-23, symbol Transistor_BJT:MMBT3904
- removed R5, R6: 33R, Resistor_SMD:R_0603_1608Metric, symbol tbraico:33R
- removed R7, R8: 22R, Resistor_SMD:R_0603_1608Metric, symbol tbraico:22R
- added R4, R6: 220R, Resistor_SMD:R_0603_1608Metric, symbol tbraico:220R
- renumbered D2 to D1, D1 to D2, R12 to R10, R13 to R11, R4 to R5, R9 to R7, R10 to R8, R11 to R9
Connections:
- net +3V3: now also D1.2 (A)
- net BAT_P: no longer C2.1, CR1.5 (I/O4), L1.1, U1.3 (VIN), U1.4 (EN/BYP)
- net GND: now also R6.2
- net at D2.1 (K): now also R6.1
- net ST: now reaches D2.2 (A), R3.2, U2.8 (ST)
- net ST: now also R4.1
- net at D1.1 (K): now also R4.2
- new net: C2.1, CR1.5 (I/O4), L1.1, U1.3 (VIN), U1.4 (EN/BYP)
Other:
- moved on the sheet: D1, D2
